Commit message: switch to glb

File: rtb-data/rtbdata/xacro/ufactory_description/lite6/urdf/lite6.urdf.xacro (robot description, xacro)
@@ -35,14 +35,14 @@
           rpy="0 0 0" />
         <geometry>
-          <mesh filename="package://ufactory_description/lite6/meshes/visual/base.stl"/>
-        </geometry>
-        <material name="${prefix}White" />
-      </visual>
-      <collision>
-        <origin
-          xyz="0 0 0"
-          rpy="0 0 0" />
-        <geometry>
-          <mesh filename="package://ufactory_description/lite6/meshes/visual/base.stl"/>
+          <mesh filename="package://ufactory_description/lite6/meshes/visual/base.glb"/>
+        </geometry>
+        <material name="${prefix}White" />
+      </visual>
+      <collision>
+        <origin
+          xyz="0 0 0"
+          rpy="0 0 0" />
+        <geometry>
+          <mesh filename="package://ufactory_description/lite6/meshes/visual/base.glb"/>
         </geometry>
       </collision>
@@ -68,14 +68,14 @@
           rpy="0 0 0" />
         <geometry>
-          <mesh filename="package://ufactory_description/lite6/meshes/visual/link1.stl"/>
-        </geometry>
-        <material name="${prefix}White" />
-      </visual>
-      <collision>
-        <origin
-          xyz="0 0 0"
-          rpy="0 0 0" />
-        <geometry>
-          <mesh filename="package://ufactory_description/lite6/meshes/visual/link1.stl"/>
+          <mesh filename="package://ufactory_description/lite6/meshes/visual/link1.glb"/>
+        </geometry>
+        <material name="${prefix}White" />
+      </visual>
+      <collision>
+        <origin
+          xyz="0 0 0"
+          rpy="0 0 0" />
+        <geometry>
+          <mesh filename="package://ufactory_description/lite6/meshes/visual/link1.glb"/>
         </geometry>
       </collision>
@@ -118,14 +118,14 @@
           rpy="0 0 0" />
         <geometry>
-           <mesh filename="package://ufactory_description/lite6/meshes/visual/link2.stl"/>
-        </geometry>
-        <material name="${prefix}White" />
-      </visual>
-      <collision>
-        <origin
-          xyz="0 0 0"
-          rpy="0 0 0" />
-        <geometry>
-           <mesh filename="package://ufactory_description/lite6/meshes/visual/link2.stl"/>
+           <mesh filename="package://ufactory_description/lite6/meshes/visual/link2.glb"/>
+        </geometry>
+        <material name="${prefix}White" />
+      </visual>
+      <collision>
+        <origin
+          xyz="0 0 0"
+          rpy="0 0 0" />
+        <geometry>
+           <mesh filename="package://ufactory_description/lite6/meshes/visual/link2.glb"/>
         </geometry>
       </collision>
@@ -168,14 +168,14 @@
           rpy="0 0 0" />
         <geometry>
-           <mesh filename="package://ufactory_description/lite6/meshes/visual/link3.stl"/>
-        </geometry>
-        <material name="${prefix}White" />
-      </visual>
-      <collision>
-        <origin
-          xyz="0 0 0"
-          rpy="0 0 0" />
-        <geometry>
-           <mesh filename="package://ufactory_description/lite6/meshes/visual/link3.stl"/>
+           <mesh filename="package://ufactory_description/lite6/meshes/visual/link3.glb"/>
+        </geometry>
+        <material name="${prefix}White" />
+      </visual>
+      <collision>
+        <origin
+          xyz="0 0 0"
+          rpy="0 0 0" />
+        <geometry>
+           <mesh filename="package://ufactory_description/lite6/meshes/visual/link3.glb"/>
         </geometry>
       </collision>
@@ -218,14 +218,14 @@
           rpy="0 0 0" />
         <geometry>
-           <mesh filename="package://ufactory_description/lite6/meshes/visual/link4.stl"/>
-        </geometry>
-        <material name="${prefix}White" />
-      </visual>
-      <collision>
-        <origin
-          xyz="0 0 0"
-          rpy="0 0 0" />
-        <geometry>
-           <mesh filename="package://ufactory_description/lite6/meshes/visual/link4.stl"/>
+           <mesh filename="package://ufactory_description/lite6/meshes/visual/link4.glb"/>
+        </geometry>
+        <material name="${prefix}White" />
+      </visual>
+      <collision>
+        <origin
+          xyz="0 0 0"
+          rpy="0 0 0" />
+        <geometry>
+           <mesh filename="package://ufactory_description/lite6/meshes/visual/link4.glb"/>
         </geometry>
       </collision>
@@ -268,14 +268,14 @@
           rpy="0 0 0" />
         <geometry>
-           <mesh filename="package://ufactory_description/lite6/meshes/visual/link5.stl"/>
-        </geometry>
-        <material name="${prefix}White" />
-      </visual>
-      <collision>
-        <origin
-          xyz="0 0 0"
-          rpy="0 0 0" />
-        <geometry>
-           <mesh filename="package://ufactory_description/lite6/meshes/visual/link5.stl"/>
+           <mesh filename="package://ufactory_description/lite6/meshes/visual/link5.glb"/>
+        </geometry>
+        <material name="${prefix}White" />
+      </visual>
+      <collision>
+        <origin
+          xyz="0 0 0"
+          rpy="0 0 0" />
+        <geometry>
+           <mesh filename="package://ufactory_description/lite6/meshes/visual/link5.glb"/>
         </geometry>
       </collision>
@@ -318,5 +318,5 @@
           rpy="0 0 0" />
         <geometry>
-           <mesh filename="package://ufactory_description/lite6/meshes/visual/link6.stl"/>
+           <mesh filename="package://ufactory_description/lite6/meshes/visual/link6.glb"/>
         </geometry>
         <material name="${prefix}Silver" />
@@ -327,5 +327,5 @@
           rpy="0 0 0" />
         <geometry>
-           <mesh filename="package://ufactory_description/lite6/meshes/visual/link6.stl"/>
+           <mesh filename="package://ufactory_description/lite6/meshes/visual/link6.glb"/>
         </geometry>
       </collision>

File: rtb-data/rtbdata/xacro/ufactory_description/lite6/urdf/lite_gripper.urdf.xacro (robot description, xacro)
@@ -33,5 +33,5 @@
         rpy="0 0 0" />
       <geometry>
-        <mesh filename="package://ufactory_description/lite6/meshes/visual/gripper_lite.stl"/>
+        <mesh filename="package://ufactory_description/lite6/meshes/visual/gripper_lite.glb"/>
       </geometry>
       <material name="White_gripper">
@@ -44,5 +44,5 @@
         rpy="0 0 0" />
       <geometry>
-        <mesh filename="package://ufactory_description/lite6/meshes/collision/gripper_lite.stl"/>
+        <mesh filename="package://ufactory_description/lite6/meshes/collision/gripper_lite.glb"/>
       </geometry>
     </collision>

File: rtb-data/rtbdata/xacro/ufactory_description/lite6/urdf/lite_gripper_pen.urdf.xacro (robot description, xacro)
@@ -33,5 +33,5 @@
         rpy="0 0 0" />
       <geometry>
-        <mesh filename="package://ufactory_description/lite6/meshes/visual/gripper_lite_pen.stl"/>
+        <mesh filename="package://ufactory_description/lite6/meshes/visual/gripper_lite_pen.glb"/>
       </geometry>
       <material name="White_gripper">
@@ -44,5 +44,5 @@
         rpy="0 0 0" />
       <geometry>
-        <mesh filename="package://ufactory_description/lite6/meshes/collision/gripper_lite_pen.stl"/>
+        <mesh filename="package://ufactory_description/lite6/meshes/collision/gripper_lite_pen.glb"/>
       </geometry>
     </collision>

Commit message: brieckiebot

File: rtb-data/rtbdata/xacro/ufactory_description/lite6/urdf/lite6.urdf.xacro (robot description, xacro)
@@ -35,14 +35,14 @@
           rpy="0 0 0" />
         <geometry>
-          <mesh filename="package://ufactory_description/lite6/meshes/visual/base.glb"/>
-        </geometry>
-        <material name="${prefix}White" />
-      </visual>
-      <collision>
-        <origin
-          xyz="0 0 0"
-          rpy="0 0 0" />
-        <geometry>
-          <mesh filename="package://ufactory_description/lite6/meshes/visual/base.glb"/>
+          <mesh filename="package://ufactory_description/lite6/meshes/visual/base.stl"/>
+        </geometry>
+        <material name="${prefix}White" />
+      </visual>
+      <collision>
+        <origin
+          xyz="0 0 0"
+          rpy="0 0 0" />
+        <geometry>
+          <mesh filename="package://ufactory_description/lite6/meshes/visual/base.stl"/>
         </geometry>
       </collision>
@@ -68,14 +68,14 @@
           rpy="0 0 0" />
         <geometry>
-          <mesh filename="package://ufactory_description/lite6/meshes/visual/link1.glb"/>
-        </geometry>
-        <material name="${prefix}White" />
-      </visual>
-      <collision>
-        <origin
-          xyz="0 0 0"
-          rpy="0 0 0" />
-        <geometry>
-          <mesh filename="package://ufactory_description/lite6/meshes/visual/link1.glb"/>
+          <mesh filename="package://ufactory_description/lite6/meshes/visual/link1.stl"/>
+        </geometry>
+        <material name="${prefix}White" />
+      </visual>
+      <collision>
+        <origin
+          xyz="0 0 0"
+          rpy="0 0 0" />
+        <geometry>
+          <mesh filename="package://ufactory_description/lite6/meshes/visual/link1.stl"/>
         </geometry>
       </collision>
@@ -118,14 +118,14 @@
           rpy="0 0 0" />
         <geometry>
-           <mesh filename="package://ufactory_description/lite6/meshes/visual/link2.glb"/>
-        </geometry>
-        <material name="${prefix}White" />
-      </visual>
-      <collision>
-        <origin
-          xyz="0 0 0"
-          rpy="0 0 0" />
-        <geometry>
-           <mesh filename="package://ufactory_description/lite6/meshes/visual/link2.glb"/>
+           <mesh filename="package://ufactory_description/lite6/meshes/visual/link2.stl"/>
+        </geometry>
+        <material name="${prefix}White" />
+      </visual>
+      <collision>
+        <origin
+          xyz="0 0 0"
+          rpy="0 0 0" />
+        <geometry>
+           <mesh filename="package://ufactory_description/lite6/meshes/visual/link2.stl"/>
         </geometry>
       </collision>
@@ -168,14 +168,14 @@
           rpy="0 0 0" />
         <geometry>
-           <mesh filename="package://ufactory_description/lite6/meshes/visual/link3.glb"/>
-        </geometry>
-        <material name="${prefix}White" />
-      </visual>
-      <collision>
-        <origin
-          xyz="0 0 0"
-          rpy="0 0 0" />
-        <geometry>
-           <mesh filename="package://ufactory_description/lite6/meshes/visual/link3.glb"/>
+           <mesh filename="package://ufactory_description/lite6/meshes/visual/link3.stl"/>
+        </geometry>
+        <material name="${prefix}White" />
+      </visual>
+      <collision>
+        <origin
+          xyz="0 0 0"
+          rpy="0 0 0" />
+        <geometry>
+           <mesh filename="package://ufactory_description/lite6/meshes/visual/link3.stl"/>
         </geometry>
       </collision>
@@ -218,14 +218,14 @@
           rpy="0 0 0" />
         <geometry>
-           <mesh filename="package://ufactory_description/lite6/meshes/visual/link4.glb"/>
-        </geometry>
-        <material name="${prefix}White" />
-      </visual>
-      <collision>
-        <origin
-          xyz="0 0 0"
-          rpy="0 0 0" />
-        <geometry>
-           <mesh filename="package://ufactory_description/lite6/meshes/visual/link4.glb"/>
+           <mesh filename="package://ufactory_description/lite6/meshes/visual/link4.stl"/>
+        </geometry>
+        <material name="${prefix}White" />
+      </visual>
+      <collision>
+        <origin
+          xyz="0 0 0"
+          rpy="0 0 0" />
+        <geometry>
+           <mesh filename="package://ufactory_description/lite6/meshes/visual/link4.stl"/>
         </geometry>
       </collision>
@@ -268,14 +268,14 @@
           rpy="0 0 0" />
         <geometry>
-           <mesh filename="package://ufactory_description/lite6/meshes/visual/link5.glb"/>
-        </geometry>
-        <material name="${prefix}White" />
-      </visual>
-      <collision>
-        <origin
-          xyz="0 0 0"
-          rpy="0 0 0" />
-        <geometry>
-           <mesh filename="package://ufactory_description/lite6/meshes/visual/link5.glb"/>
+           <mesh filename="package://ufactory_description/lite6/meshes/visual/link5.stl"/>
+        </geometry>
+        <material name="${prefix}White" />
+      </visual>
+      <collision>
+        <origin
+          xyz="0 0 0"
+          rpy="0 0 0" />
+        <geometry>
+           <mesh filename="package://ufactory_description/lite6/meshes/visual/link5.stl"/>
         </geometry>
       </collision>
@@ -318,5 +318,5 @@
           rpy="0 0 0" />
         <geometry>
-           <mesh filename="package://ufactory_description/lite6/meshes/visual/link6.glb"/>
+           <mesh filename="package://ufactory_description/lite6/meshes/visual/link6.stl"/>
         </geometry>
         <material name="${prefix}Silver" />
@@ -327,5 +327,5 @@
           rpy="0 0 0" />
         <geometry>
-           <mesh filename="package://ufactory_description/lite6/meshes/visual/link6.glb"/>
+           <mesh filename="package://ufactory_description/lite6/meshes/visual/link6.stl"/>
         </geometry>
       </collision>
